File: Kicad/DOOOPE.kicad_pcb (KiCad board)
At the start: 2 copper layers, 129.9 x 98.7 mm, 54 parts, among them J2 JST Connector, SW1 SW_PUSH, SW10 SW_PUSH, SW11 SW_PUSH, SW13 SW_PUSH, SW14 SW_PUSH, SW15 SW_PUSH, SW16 SW_PUSH, SW17 SW_PUSH, SW2 SW_PUSH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

Commit message: latest files
Parts:
- added REF**: Breakaway_Tabs, KBLib:Breakaway_Tabs, F.Cu at (24.8, 80.6)
- added kibuzzard-6465F412: G***, kibuzzard-6465F412, F.Cu at (48.6, 72.0)
- added kibuzzard-6465F412: G***, kibuzzard-6465F412, B.Cu at (48.6, 72.0)
- added kibuzzard-6465FBCD: G***, kibuzzard-6465FBCD, F.Cu at (38.9, 81.1)
- added kibuzzard-6465FBCD: G***, kibuzzard-6465FBCD, B.Cu at (38.9, 81.1)
- moved kibuzzard-643B780C 53.4 mm to (71.6, 120.4)
- moved kibuzzard-643B7841 53.4 mm to (71.6, 120.4)
- moved kibuzzard-643B7985 8.66 mm to (50.6, 72.0) (x2)
- moved G*** 2.53 mm to (85.9, 122.9)
- moved G*** 2.53 mm to (96.3, 123.2)
Connections:
- U1 pad 10: Row2 -> Col3
- U1 pad 11: Row3 -> Col2
- U1 pad 3: Col2 -> Row1
- U1 pad 4: Col3 -> Row2
- U1 pad 5: Col4 -> Row3
- U1 pad 6: Col5 -> Row0
- U1 pad 8: Row0 -> Col5
- U1 pad 9: Row1 -> Col4
Routing:
- net Row3: track 198.1 -> 134.8 mm, vias 4 -> 1
- net Row1: track 192.6 -> 163.2 mm
- net Row2: track 187.2 -> 162.6 mm, vias 4 -> 2
- net Col5: track 186.6 -> 164.5 mm, vias 2 -> 1
- net Col2: track 98.4 -> 83.7 mm, vias 3 -> 1
- net Row0: track 122.9 -> 111.0 mm, vias 4 -> 2
- net Col4: track 154.3 -> 143.4 mm, vias 2 -> 1
- net Col1: track 88.2 -> 78.4 mm
- net Col3: track 101.2 -> 95.6 mm
- net GND: track 10.4 -> 11.8 mm, vias 1 -> 16
- net Col0: track 53.4 -> 54.5 mm
Other:
- outline, holes or cut-outs redrawn
- board text added: "JLCJLCJLCJLC"
- board text removed: "-"
